Commit message: intento camara

File: panda_description/Panda/panda.xacro (robot description, xacro)
@@ -1,18 +1,18 @@
 <?xml version="1.0" ?>
-<!-- =================================================================================== -->
-<!-- |    This document was autogenerated by xacro from panda_arm_hand.urdf.xacro      | -->
-<!-- |    EDITING THIS FILE BY HAND IS NOT RECOMMENDED                                 | -->
-<!-- =================================================================================== -->
-<robot name="panda" xmlns:xacro="http://www.ros.org/wiki/xacro">
+<robot name="pandas_robot" xmlns:xacro="http://www.ros.org/wiki/xacro">
+  <xacro:property name="mesh_path" value="file:///home/starslab_go/stars_lab_ws/panda_robot/src/panda_description/Panda/meshes"/>
+  <xacro:include filename="$(find panda_description)/Panda/materials.xacro"/>
+  <xacro:include filename="$(find panda_description)/Panda/panda.gazebo"/>
+  <xacro:include filename="$(find panda_description)/Panda/macros.xacro"/>
   <link name="panda_link0">
     <visual>
       <geometry>
-        <mesh filename="/home/jingpei/Desktop/robot_pose_estimation/renderer/Panda/meshes/collision/link0.obj"/>
-      </geometry>
-      <material name="panda_white"/>
-    </visual>
-    <collision>
-      <geometry>
-        <mesh filename="/home/jingpei/Desktop/robot_pose_estimation/renderer/Panda/meshes/collision/link0.obj"/>
+        <mesh filename="${mesh_path}/collision/link0.obj"/>
+      </geometry>
+      <material name="panda_white"/>
+    </visual>
+    <collision>
+      <geometry>
+        <mesh filename="${mesh_path}/collision/link0.obj"/>
       </geometry>
       <material name="panda_white"/>
@@ -22,11 +22,11 @@
     <visual>
       <geometry>
-        <mesh filename="/home/jingpei/Desktop/robot_pose_estimation/renderer/Panda/meshes/collision/link1.obj"/>
-      </geometry>
-      <material name="panda_white"/>
-    </visual>
-    <collision>
-      <geometry>
-        <mesh filename="/home/jingpei/Desktop/robot_pose_estimation/renderer/Panda/meshes/collision/link1.obj"/>
+        <mesh filename="${mesh_path}/collision/link1.obj"/>
+      </geometry>
+      <material name="panda_white"/>
+    </visual>
+    <collision>
+      <geometry>
+        <mesh filename="${mesh_path}/collision/link1.obj"/>
       </geometry>
       <material name="panda_white"/>
@@ -44,11 +44,11 @@
     <visual>
       <geometry>
-        <mesh filename="/home/jingpei/Desktop/robot_pose_estimation/renderer/Panda/meshes/collision/link2.obj"/>
-      </geometry>
-      <material name="panda_white"/>
-    </visual>
-    <collision>
-      <geometry>
-        <mesh filename="/home/jingpei/Desktop/robot_pose_estimation/renderer/Panda/meshes/collision/link2.obj"/>
+        <mesh filename="${mesh_path}/collision/link2.obj"/>
+      </geometry>
+      <material name="panda_white"/>
+    </visual>
+    <collision>
+      <geometry>
+        <mesh filename="${mesh_path}/collision/link2.obj"/>
       </geometry>
       <material name="panda_white"/>
@@ -66,11 +66,11 @@
     <visual>
       <geometry>
-        <mesh filename="/home/jingpei/Desktop/robot_pose_estimation/renderer/Panda/meshes/collision/link3.obj"/>
-      </geometry>
-      <material name="panda_white"/>
-    </visual>
-    <collision>
-      <geometry>
-        <mesh filename="/home/jingpei/Desktop/robot_pose_estimation/renderer/Panda/meshes/collision/link3.obj"/>
+        <mesh filename="${mesh_path}/collision/link3.obj"/>
+      </geometry>
+      <material name="panda_white"/>
+    </visual>
+    <collision>
+      <geometry>
+        <mesh filename="${mesh_path}/collision/link3.obj"/>
       </geometry>
       <material name="panda_white"/>
@@ -88,11 +88,11 @@
     <visual>
       <geometry>
-        <mesh filename="/home/jingpei/Desktop/robot_pose_estimation/renderer/Panda/meshes/collision/link4.obj"/>
-      </geometry>
-      <material name="panda_white"/>
-    </visual>
-    <collision>
-      <geometry>
-        <mesh filename="/home/jingpei/Desktop/robot_pose_estimation/renderer/Panda/meshes/collision/link4.obj"/>
+        <mesh filename="${mesh_path}/collision/link4.obj"/>
+      </geometry>
+      <material name="panda_white"/>
+    </visual>
+    <collision>
+      <geometry>
+        <mesh filename="${mesh_path}/collision/link4.obj"/>
       </geometry>
       <material name="panda_white"/>
@@ -110,11 +110,11 @@
     <visual>
       <geometry>
-        <mesh filename="/home/jingpei/Desktop/robot_pose_estimation/renderer/Panda/meshes/collision/link5.obj"/>
-      </geometry>
-      <material name="panda_white"/>
-    </visual>
-    <collision>
-      <geometry>
-        <mesh filename="/home/jingpei/Desktop/robot_pose_estimation/renderer/Panda/meshes/collision/link5.obj"/>
+        <mesh filename="${mesh_path}/collision/link5.obj"/>
+      </geometry>
+      <material name="panda_white"/>
+    </visual>
+    <collision>
+      <geometry>
+        <mesh filename="${mesh_path}/collision/link5.obj"/>
       </geometry>
       <material name="panda_white"/>
@@ -132,11 +132,11 @@
     <visual>
       <geometry>
-        <mesh filename="/home/jingpei/Desktop/robot_pose_estimation/renderer/Panda/meshes/collision/link6.obj"/>
-      </geometry>
-      <material name="panda_white"/>
-    </visual>
-    <collision>
-      <geometry>
-        <mesh filename="/home/jingpei/Desktop/robot_pose_estimation/renderer/Panda/meshes/collision/link6.obj"/>
+        <mesh filename="${mesh_path}/collision/link6.obj"/>
+      </geometry>
+      <material name="panda_white"/>
+    </visual>
+    <collision>
+      <geometry>
+        <mesh filename="${mesh_path}/collision/link6.obj"/>
       </geometry>
       <material name="panda_white"/>
@@ -154,11 +154,11 @@
     <visual>
       <geometry>
-        <mesh filename="/home/jingpei/Desktop/robot_pose_estimation/renderer/Panda/meshes/collision/link7.obj"/>
-      </geometry>
-      <material name="panda_white"/>
-    </visual>
-    <collision>
-      <geometry>
-        <mesh filename="/home/jingpei/Desktop/robot_pose_estimation/renderer/Panda/meshes/collision/link7.obj"/>
+        <mesh filename="${mesh_path}/collision/link7.obj"/>
+      </geometry>
+      <material name="panda_white"/>
+    </visual>
+    <collision>
+      <geometry>
+        <mesh filename="${mesh_path}/collision/link7.obj"/>
       </geometry>
       <material name="panda_white"/>
@@ -188,11 +188,11 @@
     <visual>
       <geometry>
-        <mesh filename="/home/jingpei/Desktop/robot_pose_estimation/renderer/Panda/meshes/collision/hand.obj"/>
-      </geometry>
-      <material name="panda_white"/>
-    </visual>
-    <collision>
-      <geometry>
-        <mesh filename="/home/jingpei/Desktop/robot_pose_estimation/renderer/Panda/meshes/collision/hand.obj"/>
+        <mesh filename="${mesh_path}/collision/hand.obj"/>
+      </geometry>
+      <material name="panda_white"/>
+    </visual>
+    <collision>
+      <geometry>
+        <mesh filename="${mesh_path}/collision/hand.obj"/>
       </geometry>
       <material name="panda_white"/>
@@ -202,11 +202,11 @@
     <visual>
       <geometry>
-        <mesh filename="/home/jingpei/Desktop/robot_pose_estimation/renderer/Panda/meshes/collision/finger.obj"/>
-      </geometry>
-      <material name="panda_white"/>
-    </visual>
-    <collision>
-      <geometry>
-        <mesh filename="/home/jingpei/Desktop/robot_pose_estimation/renderer/Panda/meshes/collision/finger.obj"/>
+        <mesh filename="${mesh_path}/collision/finger.obj"/>
+      </geometry>
+      <material name="panda_white"/>
+    </visual>
+    <collision>
+      <geometry>
+        <mesh filename="${mesh_path}/collision/finger.obj"/>
       </geometry>
       <material name="panda_white"/>
@@ -217,5 +217,5 @@
       <origin rpy="0 0 3.14159265359" xyz="0 0 0"/>
       <geometry>
-        <mesh filename="/home/jingpei/Desktop/robot_pose_estimation/renderer/Panda/meshes/collision/finger.obj"/>
+        <mesh filename="${mesh_path}/collision/finger.obj"/>
       </geometry>
       <material name="panda_white"/>
@@ -224,5 +224,5 @@
       <origin rpy="0 0 3.14159265359" xyz="0 0 0"/>
       <geometry>
-        <mesh filename="/home/jingpei/Desktop/robot_pose_estimation/renderer/Panda/meshes/collision/finger.obj"/>
+        <mesh filename="${mesh_path}/collision/finger.obj"/>
       </geometry>
       <material name="panda_white"/>
@@ -247,3 +247,28 @@
     <color rgba="1. 1. 1. 1."/>
   </material>
+  <link name="sensor_laser">
+    <inertial>
+      <origin xyz="0 0 0" rpy="0 0 0" />
+      <mass value="1" />
+      <xacro:cylinder_inertia mass="1" r="0.05" l="0.1" />
+    </inertial>
+    <visual>
+      <origin xyz="0 0 0" rpy="0 0 0" />
+      <geometry>
+        <cylinder radius="0.05" length="0.1"/>
+      </geometry>
+      <material name="white" />
+    </visual>
+    <collision>
+      <origin xyz="0 0 0" rpy="0 0 0"/>
+      <geometry>
+        <cylinder radius="0.05" length="0.1"/>
+      </geometry>
+    </collision>
+  </link>
+  <joint name="joint_sensor_laser" type="fixed">
+    <origin xyz="0.26 0 0.0" rpy="0 0 0"/>
+    <parent link="panda_link0"/>
+    <child link="sensor_laser"/>
+  </joint>
 </robot>
