Commit message: dataset, inertia updates, README file for camera shots automation

File: panda_description/urdf/visuals.xacro (robot description, xacro)
@@ -3,5 +3,5 @@
     <link name="panda_link0">
     <inertial>
-      <mass value="1" />
+      <mass value="0.1" />
       <origin xyz="0 0 0" rpy="0 0 0"/>
       <inertia ixx="0.05" ixy="0" ixz="0" iyy="0.05" iyz="0" izz="0.05" />
@@ -21,5 +21,5 @@
   <link name="panda_link1">
     <inertial>
-      <mass value="1" />
+      <mass value="0.1" />
       <origin xyz="0 0 0" rpy="0 0 0"/>
       <inertia ixx="0.05" ixy="0" ixz="0" iyy="0.05" iyz="0" izz="0.05" />
@@ -49,5 +49,5 @@
   <link name="panda_link2">
     <inertial>
-      <mass value="1" />
+      <mass value="0.1" />
       <origin xyz="0 0 0" rpy="0 0 0"/>
       <inertia ixx="0.05" ixy="0" ixz="0" iyy="0.05" iyz="0" izz="0.05" />
@@ -77,5 +77,5 @@
   <link name="panda_link3">
     <inertial>
-      <mass value="1" />
+      <mass value="0.1" />
       <origin xyz="0 0 0" rpy="0 0 0"/>
       <inertia ixx="0.05" ixy="0" ixz="0" iyy="0.05" iyz="0" izz="0.05" />
@@ -105,5 +105,5 @@
   <link name="panda_link4">
     <inertial>
-      <mass value="1" />
+      <mass value="0.1" />
       <origin xyz="0 0 0" rpy="0 0 0"/>
       <inertia ixx="0.05" ixy="0" ixz="0" iyy="0.05" iyz="0" izz="0.05" />
@@ -133,5 +133,5 @@
   <link name="panda_link5">
     <inertial>
-      <mass value="1" />
+      <mass value="0.1" />
       <origin xyz="0 0 0" rpy="0 0 0"/>
       <inertia ixx="0.05" ixy="0" ixz="0" iyy="0.05" iyz="0" izz="0.05" />
@@ -161,5 +161,5 @@
   <link name="panda_link6">
     <inertial>
-      <mass value="1" />
+      <mass value="0.1" />
       <origin xyz="0 0 0" rpy="0 0 0"/>
       <inertia ixx="0.05" ixy="0" ixz="0" iyy="0.05" iyz="0" izz="0.05" />
@@ -189,5 +189,5 @@
   <link name="panda_link7">
     <inertial>
-      <mass value="1" />
+      <mass value="0.1" />
       <origin xyz="0 0 0" rpy="0 0 0"/>
       <inertia ixx="0.05" ixy="0" ixz="0" iyy="0.05" iyz="0" izz="0.05" />
@@ -224,5 +224,5 @@
   <link name="panda_hand">
     <inertial>
-      <mass value="1" />
+      <mass value="0.1" />
       <origin xyz="0 0 0" rpy="0 0 0"/>
       <inertia ixx="0.05" ixy="0" ixz="0" iyy="0.05" iyz="0" izz="0.05" />
@@ -249,5 +249,5 @@
   <link name="panda_leftfinger">
     <inertial>
-      <mass value="1" />
+      <mass value="0.1" />
       <origin xyz="0 0 0" rpy="0 0 0"/>
       <inertia ixx="0.05" ixy="0" ixz="0" iyy="0.05" iyz="0" izz="0.05" />
@@ -269,5 +269,5 @@
   <link name="panda_rightfinger">
     <inertial>
-      <mass value="1" />
+      <mass value="0.1" />
       <origin xyz="0 0 0" rpy="0 0 0"/>
       <inertia ixx="0.05" ixy="0" ixz="0" iyy="0.05" iyz="0" izz="0.05" />
